Commit message: Add trash bins

File: trash_bin.urdf (robot description, URDF)
Before this commit: robot bin, 1 links, 0 joints
Links:
- link bin_body: geometry collision box size=0.01 2.5 0.17; collision box size=0.01 2.5 0.17

Commit message: Add bins (Recycling & trash)

File: trash_bin.urdf (robot description, URDF)
Before this commit: robot trash_bin, 1 links, 0 joints
Links:
- link bin_body: geometry collision box size=0.01 0.58 0.17; collision box size=0.01 0.58 0.17
