Commit message: generated variant urdfs

File: assets/urdf/ycb_variants/002_master_chef_can_var0.urdf (robot description, URDF)
Before this commit: robot 002_master_chef_can, 1 links, 0 joints
Links:
- link _name: geometry collision mesh filename=ycb/002_master_chef_can/google_16k/textured_vhacd.obj scale=9.724865988233471 10.380054608094902 9.968420743203467; visual mesh filename=ycb/002_master_chef_can/google_16k/textured.obj scale=10.270544325328002 10.219819868732742 9.569177898699209

File: assets/urdf/ycb_variants/002_master_chef_can_var1.urdf (robot description, URDF)
Before this commit: robot 002_master_chef_can, 1 links, 0 joints
Links:
- link _name: geometry collision mesh filename=ycb/002_master_chef_can/google_16k/textured_vhacd.obj scale=9.84022020183337 10.03083370450038 9.75865547416592; visual mesh filename=ycb/002_master_chef_can/google_16k/textured.obj scale=10.193326759986844 10.360909022772502 10.010487465166483

File: assets/urdf/ycb_variants/002_master_chef_can_var2.urdf (robot description, URDF)
Before this commit: robot 002_master_chef_can, 1 links, 0 joints
Links:
- link _name: geometry collision mesh filename=ycb/002_master_chef_can/google_16k/textured_vhacd.obj scale=9.993321341237756 10.48529514498121 9.990069952964207; visual mesh filename=ycb/002_master_chef_can/google_16k/textured.obj scale=10.14485539972273 10.379950423652978 10.133420703533389

File: assets/urdf/ycb_variants/002_master_chef_can_var3.urdf (robot description, URDF)
Before this commit: robot 002_master_chef_can, 1 links, 0 joints
Links:
- link _name: geometry collision mesh filename=ycb/002_master_chef_can/google_16k/textured_vhacd.obj scale=10.240792237950336 10.237772626424297 9.509067161787508; visual mesh filename=ycb/002_master_chef_can/google_16k/textured.obj scale=9.815031218139264 10.284640088447706 9.985610970145405

File: assets/urdf/ycb_variants/002_master_chef_can_var4.urdf (robot description, URDF)
Before this commit: robot 002_master_chef_can, 1 links, 0 joints
Links:
- link _name: geometry collision mesh filename=ycb/002_master_chef_can/google_16k/textured_vhacd.obj scale=10.454920955021342 10.46357439929238 9.487351342697032; visual mesh filename=ycb/002_master_chef_can/google_16k/textured.obj scale=9.786527504052241 10.108146319873962 9.588057371788969

Commit message: change used urdfs

File: assets/urdf/ycb_variants/002_master_chef_can_var0.urdf (robot description, URDF)
Before this commit: robot 002_master_chef_can, 1 links, 0 joints
Links:
- link _name: geometry collision mesh filename=ycb/002_master_chef_can/google_16k/textured_vhacd.obj scale=9.936228766515855 9.629753430175853 9.714962682259088; visual mesh filename=ycb/002_master_chef_can/google_16k/textured.obj scale=10.187791332117728 10.110402762333006 10.47500735506192

File: assets/urdf/ycb_variants/002_master_chef_can_var1.urdf (robot description, URDF)
Before this commit: robot 002_master_chef_can, 1 links, 0 joints
Links:
- link _name: geometry collision mesh filename=ycb/002_master_chef_can/google_16k/textured_vhacd.obj scale=10.06456696324358 9.158699020999517 9.952588200325234; visual mesh filename=ycb/002_master_chef_can/google_16k/textured.obj scale=10.579918147012284 9.766764261647605 10.456101424308814

File: assets/urdf/ycb_variants/002_master_chef_can_var2.urdf (robot description, URDF)
Before this commit: robot 002_master_chef_can, 1 links, 0 joints
Links:
- link _name: geometry collision mesh filename=ycb/002_master_chef_can/google_16k/textured_vhacd.obj scale=10.134507306631818 8.823600331718934 9.517950532807376; visual mesh filename=ycb/002_master_chef_can/google_16k/textured.obj scale=10.59226400768065 9.320843750621405 10.005601195962049

File: assets/urdf/ycb_variants/002_master_chef_can_var3.urdf (robot description, URDF)
Before this commit: robot 002_master_chef_can, 1 links, 0 joints
Links:
- link _name: geometry collision mesh filename=ycb/002_master_chef_can/google_16k/textured_vhacd.obj scale=10.611558623061947 8.908159766973306 9.884011827656176; visual mesh filename=ycb/002_master_chef_can/google_16k/textured.obj scale=10.570333758126212 9.662838664281544 9.627302127224436

File: assets/urdf/ycb_variants/002_master_chef_can_var4.urdf (robot description, URDF)
Before this commit: robot 002_master_chef_can, 1 links, 0 joints
Links:
- link _name: geometry collision mesh filename=ycb/002_master_chef_can/google_16k/textured_vhacd.obj scale=10.314673547304027 8.956135405068947 10.274556021218865; visual mesh filename=ycb/002_master_chef_can/google_16k/textured.obj scale=10.174008795602711 9.468679376491805 9.750010015372352

File: assets/urdf/ycb_variants/003_cracker_box_var0.urdf (robot description, URDF)
Before this commit: robot 003_cracker_box, 1 links, 0 joints
Links:
- link _name: geometry collision mesh filename=ycb/003_cracker_box/google_16k/textured_vhacd.obj scale=9.715125918016078 10.001600964922046 10.398288784368104; visual mesh filename=ycb/003_cracker_box/google_16k/textured.obj scale=10.4071993776009 10.145838355683445 10.375821851494432

File: assets/urdf/ycb_variants/003_cracker_box_var1.urdf (robot description, URDF)
Before this commit: robot 003_cracker_box, 1 links, 0 joints
Links:
- link _name: geometry collision mesh filename=ycb/003_cracker_box/google_16k/textured_vhacd.obj scale=9.998187668600709 10.1260092569737 10.50030740571755; visual mesh filename=ycb/003_cracker_box/google_16k/textured.obj scale=9.945079618941225 10.640363715754052 10.308803755081174

File: assets/urdf/ycb_variants/003_cracker_box_var2.urdf (robot description, URDF)
Before this commit: robot 003_cracker_box, 1 links, 0 joints
Links:
- link _name: geometry collision mesh filename=ycb/003_cracker_box/google_16k/textured_vhacd.obj scale=10.301309265811954 10.078863486583849 10.199333045365993; visual mesh filename=ycb/003_cracker_box/google_16k/textured.obj scale=9.687741454451247 11.087657749106137 10.7729191805945

File: assets/urdf/ycb_variants/003_cracker_box_var3.urdf (robot description, URDF)
Before this commit: robot 003_cracker_box, 1 links, 0 joints
Links:
- link _name: geometry collision mesh filename=ycb/003_cracker_box/google_16k/textured_vhacd.obj scale=9.982891188253033 9.721241566338087 10.398802875398147; visual mesh filename=ycb/003_cracker_box/google_16k/textured.obj scale=9.530004827604113 11.376992560245714 11.294268631734328

File: assets/urdf/ycb_variants/003_cracker_box_var4.urdf (robot description, URDF)
Before this commit: robot 003_cracker_box, 1 links, 0 joints
Links:
- link _name: geometry collision mesh filename=ycb/003_cracker_box/google_16k/textured_vhacd.obj scale=9.543373400608283 9.328651292919862 10.803417814271192; visual mesh filename=ycb/003_cracker_box/google_16k/textured.obj scale=9.812918853006385 11.36915282224951 11.769718505584498

File: assets/urdf/ycb_variants/004_sugar_box_var0.urdf (robot description, URDF)
Before this commit: robot 004_sugar_box, 1 links, 0 joints
Links:
- link _name: geometry collision mesh filename=ycb/004_sugar_box/google_16k/textured_vhacd.obj scale=9.88303861693203 9.510639703864074 10.322356367353311; visual mesh filename=ycb/004_sugar_box/google_16k/textured.obj scale=9.883521688670477 10.412893814174385 10.198496394465796

File: assets/urdf/ycb_variants/004_sugar_box_var1.urdf (robot description, URDF)
Before this commit: robot 004_sugar_box, 1 links, 0 joints
Links:
- link _name: geometry collision mesh filename=ycb/004_sugar_box/google_16k/textured_vhacd.obj scale=9.717294690893457 9.709042056372523 10.61333402129244; visual mesh filename=ycb/004_sugar_box/google_16k/textured.obj scale=10.088077352712572 9.934517202303047 9.713303464535446

File: assets/urdf/ycb_variants/004_sugar_box_var2.urdf (robot description, URDF)
Before this commit: robot 004_sugar_box, 1 links, 0 joints
Links:
- link _name: geometry collision mesh filename=ycb/004_sugar_box/google_16k/textured_vhacd.obj scale=10.082548215442717 9.742836507537037 10.843575933409323; visual mesh filename=ycb/004_sugar_box/google_16k/textured.obj scale=9.67364986828693 10.365187104751545 9.286034460337069

File: assets/urdf/ycb_variants/004_sugar_box_var3.urdf (robot description, URDF)
Before this commit: robot 004_sugar_box, 1 links, 0 joints
Links:
- link _name: geometry collision mesh filename=ycb/004_sugar_box/google_16k/textured_vhacd.obj scale=10.079239343127755 9.934964691895216 10.440684675902038; visual mesh filename=ycb/004_sugar_box/google_16k/textured.obj scale=9.272578186763187 10.47560083912179 8.827467657691823

File: assets/urdf/ycb_variants/004_sugar_box_var4.urdf (robot description, URDF)
Before this commit: robot 004_sugar_box, 1 links, 0 joints
Links:
- link _name: geometry collision mesh filename=ycb/004_sugar_box/google_16k/textured_vhacd.obj scale=10.274485491471513 9.867787213635317 10.227800705513587; visual mesh filename=ycb/004_sugar_box/google_16k/textured.obj scale=9.707682717035226 10.586103141800365 8.985471281031515

File: assets/urdf/ycb_variants/005_tomato_soup_can_var0.urdf (robot description, URDF)
Before this commit: robot 005_tomato_soup_can, 1 links, 0 joints
Links:
- link _name: geometry collision mesh filename=ycb/005_tomato_soup_can/google_16k/textured_vhacd.obj scale=9.777224829291063 9.533915433259835 10.299905025533015; visual mesh filename=ycb/005_tomato_soup_can/google_16k/textured.obj scale=10.103759153749632 10.293912738378673 10.025830681335375

File: assets/urdf/ycb_variants/005_tomato_soup_can_var1.urdf (robot description, URDF)
Before this commit: robot 005_tomato_soup_can, 1 links, 0 joints
Links:
- link _name: geometry collision mesh filename=ycb/005_tomato_soup_can/google_16k/textured_vhacd.obj scale=9.676979279864307 9.98831116608408 10.376824762079599; visual mesh filename=ycb/005_tomato_soup_can/google_16k/textured.obj scale=10.177645928272167 10.130037541523901 10.27918359907286

File: assets/urdf/ycb_variants/005_tomato_soup_can_var2.urdf (robot description, URDF)
Before this commit: robot 005_tomato_soup_can, 1 links, 0 joints
Links:
- link _name: geometry collision mesh filename=ycb/005_tomato_soup_can/google_16k/textured_vhacd.obj scale=9.764070778456045 10.407937880166234 9.954138455211114; visual mesh filename=ycb/005_tomato_soup_can/google_16k/textured.obj scale=10.439093331643376 9.753409442899983 10.082294088955985

File: assets/urdf/ycb_variants/005_tomato_soup_can_var3.urdf (robot description, URDF)
Before this commit: robot 005_tomato_soup_can, 1 links, 0 joints
Links:
- link _name: geometry collision mesh filename=ycb/005_tomato_soup_can/google_16k/textured_vhacd.obj scale=9.802037806166611 10.084271428564538 10.007737635289256; visual mesh filename=ycb/005_tomato_soup_can/google_16k/textured.obj scale=10.221193627097119 9.961617386016579 10.218242846872842

File: assets/urdf/ycb_variants/005_tomato_soup_can_var4.urdf (robot description, URDF)
Before this commit: robot 005_tomato_soup_can, 1 links, 0 joints
Links:
- link _name: geometry collision mesh filename=ycb/005_tomato_soup_can/google_16k/textured_vhacd.obj scale=10.01391934360112 9.702931865017138 9.625848435138932; visual mesh filename=ycb/005_tomato_soup_can/google_16k/textured.obj scale=10.390066943168906 10.177361611999679 9.877151406441511
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